File: design/kicad/main_board/main_board.kicad_sch (KiCad schematic)
At the start: 6 parts, among them J1 DisplayHeader, J2 Ultrasonic_USB, J3 Ultrasonic_Header, J4 PicoHeader_1, J5 PicoHeader_2, U1 Pico

Commit message: kicad footprints allocated
Parts:
- J1: footprint (none) -> Connector_PinHeader_2.54mm:PinHeader_1x05_P2.54mm_Vertical
- J2: footprint (none) -> Connector_USB:USB_A_Molex_67643_Horizontal
- J3: footprint (none) -> Connector_PinHeader_2.54mm:PinHeader_1x04_P2.54mm_Vertical
- J4, J5: footprint (none) -> Connector_PinHeader_2.54mm:PinHeader_1x20_P2.54mm_Vertical
Changed lines of the file:
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@@
 (kicad_sch (version 20230121) (generator eeschema)
   (paper "A4")
+  (wire (pts (xy 29.21 58.42) (xy 29.21 59.69))
+    (stroke (width 0) (type default))
+  )
+  (wire (pts (xy 30.48 59.69) (xy 29.21 59.69))
+    (stroke (width 0) (type default))
+  )
   (symbol (lib_id "MCU_RaspberryPi_and_Boards:Pico") (at 71.12 48.26 0) (unit 1)
     (in_bom yes) (on_board yes) (dnp no) (fields_autoplaced)
@@
       (effects (font (size 1.27 1.27)) (justify left))
     )
-    (property "Footprint" "" (at 106.68 99.06 0)
+    (property "Footprint" "Connector_PinHeader_2.54mm:PinHeader_1x20_P2.54mm_Vertical" (at 106.68 99.06 0)
       (effects (font (size 1.27 1.27)) hide)
     )
@@
       (effects (font (size 1.27 1.27)) (justify left))
     )
-    (property "Footprint" "" (at 113.03 53.34 0)
+    (property "Footprint" "Connector_PinHeader_2.54mm:PinHeader_1x05_P2.54mm_Vertical" (at 113.03 53.34 0)
       (effects (font (size 1.27 1.27)) hide)
     )
@@
       (effects (font (size 1.27 1.27)))
     )
-    (property "Footprint" "" (at 31.75 39.37 0)
+    (property "Footprint" "Connector_USB:USB_A_Molex_67643_Horizontal" (at 31.75 39.37 0)
       (effects (font (size 1.27 1.27)) hide)
     )
@@
       (effects (font (size 1.27 1.27)))
     )
-    (property "Footprint" "" (at 25.4 59.69 0)
+    (property "Footprint" "Connector_PinHeader_2.54mm:PinHeader_1x04_P2.54mm_Vertical" (at 25.4 59.69 0)
       (effects (font (size 1.27 1.27)) hide)
     )
@@
       (effects (font (size 1.27 1.27)) (justify left))
     )
-    (property "Footprint" "" (at 46.99 97.79 0)
-      (effects (font (size 1.27 1.27)) hide)
-    )
+    (property "Footprint" "Connector_PinHeader_2.54mm:PinHeader_1x20_P2.54mm_Vertical" (at 46.99 97.79 0)
+      (effects (font (size 1.27 1.27)) hide)
+    )
